Commit message: Added RECIPES.md

File: ws/src/indoor_1/urdf/example_robot.urdf (robot description, URDF)
Before this commit: robot example_robot, 4 links, 3 joints
Links:
- added link base_footprint
Joints:
- added joint base_footprint_to_chassis_joint: type fixed, parent base_footprint, child chassis, origin xyz=0 0 0.4 rpy=0 0 0
