Commit message: Simulation partial update; edited .xacro etc

File: ws/src/indoor_1/urdf/clown_car.urdf.xacro (robot description, xacro)
@@ -1,9 +1,23 @@
 <?xml version="1.0"?>
-<robot name="clown_car">
+<robot name="clown_car" xmlns:xacro="http://ros.org/wiki/xacro">
+    <!-- Define robot constants -->
+    <xacro:property name="base_width" value="1.0" />
+    <xacro:property name="base_length" value="2.0" />
+    <xacro:property name="base_height" value="0.5" />
+    <xacro:property name="wheel_radius" value="0.4" />
+    <xacro:property name="wheel_width" value="0.2" />
+    <xacro:property name="wheel_ygap" value="1.2" />
+    <xacro:property name="wheel_zoff" value="0.0" />
+    <xacro:property name="wheel_xoff" value="-0.5" />
+    <xacro:property name="caster_xoff" value="0.8" />
+    <xacro:property name="caster_zoff" value="-0.2" />
+    <xacro:property name="imu_zoff" value="0.15" />
+    <xacro:property name="lidar_zoff" value="0.25" />
+    <xacro:property name="chassis_zoff" value="0.4" />
     <link name="base_footprint" />
     <joint name="base_footprint_to_chassis_joint" type="fixed">
         <parent link="base_footprint" />
         <child link="chassis" />
-        <origin xyz="0 0 0.4" rpy="0 0 0" />
+        <origin xyz="0 0 ${chassis_zoff}" rpy="0 0 0" />
     </joint>
     <link name="chassis">
@@ -16,5 +30,5 @@
             <origin xyz="0 0 0" rpy="0 0 0" />
             <geometry>
-                <box size="2.0 1.0 0.5" />
+                <box size="${base_length} ${base_width} ${base_height}" />
             </geometry>
         </visual>
@@ -22,5 +36,5 @@
             <origin xyz="0 0 0" rpy="0 0 0" />
             <geometry>
-                <box size="2.0 1.0 0.5" />
+                <box size="${base_length} ${base_width} ${base_height}" />
             </geometry>
         </collision>
@@ -30,5 +44,5 @@
         <parent link="chassis" />
         <child link="imu_link" />
-        <origin xyz="0 0 0.15" rpy="0 0 0" />
+        <origin xyz="0 0 ${imu_zoff}" rpy="0 0 0" />
     </joint>
     <link name="lidar_link" />
@@ -36,5 +50,5 @@
         <parent link="chassis" />
         <child link="lidar_link" />
-        <origin xyz="0 0 0.25" rpy="0 0 0" />
+        <origin xyz="0 0 ${lidar_zoff}" rpy="0 0 0" />
     </joint>
     <gazebo reference="imu_link">
@@ -88,5 +102,5 @@
             <origin xyz="0 0 0" rpy="0 0 0" />
             <geometry>
-                <cylinder radius="0.4" length="0.2" />
+                <cylinder radius="${wheel_radius}" length="${wheel_width}" />
             </geometry>
         </visual>
@@ -94,10 +108,10 @@
             <origin xyz="0 0 0" rpy="0 0 0" />
             <geometry>
-                <cylinder radius="0.4" length="0.2" />
+                <cylinder radius="${wheel_radius}" length="${wheel_width}" />
             </geometry>
         </collision>
     </link>
     <joint name="left_wheel_joint" type="continuous">
-        <origin xyz="-0.5 0.6 0" rpy="-1.5707 0 0" />
+        <origin xyz="${wheel_xoff} ${wheel_ygap / 2.0} ${wheel_zoff}" rpy="-1.5707 0 0" />
         <parent link="chassis" />
         <child link="left_wheel" />
@@ -116,5 +130,5 @@
             <origin xyz="0 0 0" rpy="0 0 0" />
             <geometry>
-                <cylinder radius="0.4" length="0.2" />
+                <cylinder radius="${wheel_radius}" length="${wheel_width}" />
             </geometry>
         </visual>
@@ -122,10 +136,10 @@
             <origin xyz="0 0 0" rpy="0 0 0" />
             <geometry>
-                <cylinder radius="0.4" length="0.2" />
+                <cylinder radius="${wheel_radius}" length="${wheel_width}" />
             </geometry>
         </collision>
     </link>
     <joint name="right_wheel_joint" type="continuous">
-        <origin xyz="-0.5 -0.6 0" rpy="-1.5707 0 0" />
+        <origin xyz="${wheel_xoff} ${-wheel_ygap / 2.0} ${wheel_zoff}" rpy="-1.5707 0 0" />
         <parent link="chassis" />
         <child link="right_wheel" />
@@ -155,5 +169,5 @@
     </link>
     <joint name="caster_wheel" type="continuous">
-        <origin xyz="0.8 0 -0.2" rpy="0 0 0" />
+        <origin xyz="${caster_xoff} 0 ${caster_zoff}" rpy="0 0 0" />
         <parent link="chassis" />
         <child link="caster" />
@@ -171,6 +185,6 @@
             <left_joint>left_wheel_joint</left_joint>
             <right_joint>right_wheel_joint</right_joint>
-            <wheel_separation>1.2</wheel_separation>
-            <wheel_radius>0.4</wheel_radius>
+            <wheel_separation>${wheel_ygap}</wheel_separation>
+            <wheel_radius>${wheel_radius}</wheel_radius>
             <odom_publish_frequency>1</odom_publish_frequency>
             <topic>cmd_vel</topic>

Commit message: Updated files, fixed missing frames, improved . .xacro file

File: ws/src/indoor_1/urdf/clown_car.urdf.xacro (robot description, xacro)
@@ -14,12 +14,12 @@
     <xacro:property name="imu_zoff" value="0.15" />
     <xacro:property name="lidar_zoff" value="0.25" />
-    <xacro:property name="chassis_zoff" value="0.4" />
+    <xacro:property name="base_link_zoff" value="0.4" />
     <link name="base_footprint" />
-    <joint name="base_footprint_to_chassis_joint" type="fixed">
+    <joint name="base_footprint_joint" type="fixed">
         <parent link="base_footprint" />
-        <child link="chassis" />
-        <origin xyz="0 0 ${chassis_zoff}" rpy="0 0 0" />
-    </joint>
-    <link name="chassis">
+        <child link="base_link" />
+        <origin xyz="0 0 ${base_link_zoff}" rpy="0 0 0" />
+    </joint>
+    <link name="base_link">
         <inertial>
             <origin xyz="0 0 0" rpy="0 0 0" />
@@ -42,5 +42,5 @@
     <link name="imu_link" />
     <joint name="imu_joint" type="fixed">
-        <parent link="chassis" />
+        <parent link="base_link" />
         <child link="imu_link" />
         <origin xyz="0 0 ${imu_zoff}" rpy="0 0 0" />
@@ -48,5 +48,5 @@
     <link name="lidar_link" />
     <joint name="lidar_joint" type="fixed">
-        <parent link="chassis" />
+        <parent link="base_link" />
         <child link="lidar_link" />
         <origin xyz="0 0 ${lidar_zoff}" rpy="0 0 0" />
@@ -55,7 +55,8 @@
         <sensor name="imu_sensor" type="imu">
             <always_on>1</always_on>
-            <update_rate>1</update_rate>
+            <update_rate>100</update_rate>
             <visualize>true</visualize>
             <topic>/imu</topic>
+            <gz_frame_id>imu_link</gz_frame_id>
         </sensor>
     </gazebo>
@@ -63,8 +64,7 @@
         <material>Gazebo/Blue</material>
         <sensor name="gpu_lidar" type="gpu_lidar">
+            <gz_frame_id>lidar_link</gz_frame_id>
             <pose>0 0 0 0 0 0</pose>
-            <!-- <topic>lidar</topic> -->
-            <laser_topic>lidar/scan</laser_topic>
-            <point_cloud_topic>lidar/points</point_cloud_topic>
+            <topic>lidar</topic>
             <update_rate>10</update_rate>
             <ray>
@@ -114,5 +114,5 @@
     <joint name="left_wheel_joint" type="continuous">
         <origin xyz="${wheel_xoff} ${wheel_ygap / 2.0} ${wheel_zoff}" rpy="-1.5707 0 0" />
-        <parent link="chassis" />
+        <parent link="base_link" />
         <child link="left_wheel" />
         <axis xyz="0 0 1" />
@@ -142,5 +142,5 @@
     <joint name="right_wheel_joint" type="continuous">
         <origin xyz="${wheel_xoff} ${-wheel_ygap / 2.0} ${wheel_zoff}" rpy="-1.5707 0 0" />
-        <parent link="chassis" />
+        <parent link="base_link" />
         <child link="right_wheel" />
         <axis xyz="0 0 1" />
@@ -170,7 +170,7 @@
     <joint name="caster_wheel" type="continuous">
         <origin xyz="${caster_xoff} 0 ${caster_zoff}" rpy="0 0 0" />
-        <parent link="chassis" />
+        <parent link="base_link" />
         <child link="caster" />
-        <axis xyz="1 1 1" />
+        <axis xyz="0 0 1" />
     </joint>
     <gazebo reference="caster">
@@ -187,5 +187,5 @@
             <wheel_separation>${wheel_ygap}</wheel_separation>
             <wheel_radius>${wheel_radius}</wheel_radius>
-            <odom_publish_frequency>1</odom_publish_frequency>
+            <odom_publish_frequency>10</odom_publish_frequency>
             <topic>cmd_vel</topic>
             <frame_id>odom</frame_id>
@@ -193,3 +193,12 @@
         </plugin>
     </gazebo>
+    <gazebo>
+        <plugin
+            filename="gz-sim-joint-state-publisher-system"
+            name="gz::sim::systems::JointStatePublisher">
+            <joint_name>left_wheel_joint</joint_name>
+            <joint_name>right_wheel_joint</joint_name>
+            <joint_name>caster_wheel</joint_name>
+        </plugin>
+    </gazebo>
 </robot>
