Commit message: Added robot, bridged gz topics, preparing for SLAM

File: ws/src/indoor_1/urdf/clown_car.urdf.xacro (robot description, xacro)
@@ -15,5 +15,10 @@
     <xacro:property name="lidar_zoff" value="0.25" />
     <xacro:property name="base_link_zoff" value="0.4" />
-    <link name="base_footprint" />
+    <link name="base_footprint">
+        <inertial>
+        <mass value="0.01" />
+        <inertia ixx="0.0001" ixy="0.0" ixz="0.0" iyy="0.0001" iyz="0.0" izz="0.0001" />
+        </inertial>
+    </link>
     <joint name="base_footprint_joint" type="fixed">
         <parent link="base_footprint" />
@@ -72,5 +77,5 @@
                     <horizontal>
                         <samples>640</samples>
-                        <resolution>1</resolution>
+                        <resolution>10</resolution>
                         <min_angle>-1.396263</min_angle>
                         <max_angle>1.396263</max_angle>
@@ -188,5 +193,5 @@
             <wheel_radius>${wheel_radius}</wheel_radius>
             <odom_publish_frequency>10</odom_publish_frequency>
-            <topic>cmd_vel</topic>
+            <topic>/cmd_vel</topic>
             <frame_id>odom</frame_id>
             <child_frame_id>base_footprint</child_frame_id>
